File: WireMonitor.kicad_pcb (KiCad board)
At the start: 2 copper layers, 18.8 x 6.1 mm, 5 parts, among them J1 2191160161, U1 INA4180A1, U2 INA4180A1, U3 INA4180A1

Commit message: schematic
Parts:
- removed U1 (x2), U2, U3: INA4180A1, Package_SO:TSSOP-14_4.4x5mm_P0.65mm
- moved J1 13.3 mm to (155.3, 77.3)
Connections:
- J1 pad P1: unconnected-(J1-PadP1) -> /L1
- J1 pad P2: unconnected-(J1-PadP2) -> /L2
- J1 pad P3: unconnected-(J1-PadP3) -> /L3
- J1 pad P4: unconnected-(J1-PadP4) -> /L4
- J1 pad P5: unconnected-(J1-PadP5) -> /L5
- J1 pad P6: unconnected-(J1-PadP6) -> /L6
